File: hw/pcb/pc_side/serial_optical_adaptor.kicad_pcb (KiCad board)
At the start: 2 copper layers, 23.2 x 58.8 mm, 13 parts, among them P3 CONN_01X04, U1 LM393, U2 CP2102

Commit message: 
Parts:
- removed P3: CONN_01X04, Pin_Headers:Pin_Header_Straight_1x04
- added P1: USB_B, Connect:USB_B, F.Cu at (97.0, 113.8)
- added P2: CONN_01X06, Pin_Headers:Pin_Header_Straight_1x06, F.Cu at (89.7, 101.5)
Connections:
- D2 pad 2: /VCC -> /Vdd
- R2 pad 1: /VCC -> /Vdd
- R3 pad 1: /VCC -> /Vdd
- R4 pad 1: /VCC -> /Vdd
- R6 pad 1: /VCC -> /Vdd
- U1 pad 8: /VCC -> /Vdd
- U2 pad 29: (no net) -> /GND
- U2 pad 7: /VCC -> /Vbus
- U2 pad 8: /VCC -> /Vbus
Routing:
- net /Vdd: track 0.00 -> 91.0 mm
- net /VCC: track 56.3 -> 3.30 mm
- net /GND: track 6.71 -> 17.5 mm
- net /Vbus: track 0.00 -> 4.98 mm
- net /TX: track 25.4 -> 24.9 mm
- net /RX: track 71.4 -> 71.9 mm
