File: hw/pcb/pc_side/serial_optical_adaptor.sch (KiCad schematic (older format))
At the start: 13 parts, among them P1 USB_B, P2 CONN_01X06, U1 LM393, U2 CP2102

Commit message: 123
Other:
- note removed: "FIBER OPTIC\nCABLE"
Changed lines of the file:
@@
 Text Notes 1700 650  0    60   ~ 0
 TRANSMITTER
-Text Notes 3050 1600 0    60   ~ 0
-FIBER OPTIC\nCABLE
 $Comp
 L IF-E97 D1
@@
 	5900 1950 5900 750
 Connection ~ 5900 750
-Wire Bus Line
-	2850 1450 3000 1450
-Wire Bus Line
-	2850 1550 3000 1550
-Wire Bus Line
-	3650 1450 3800 1450
-Wire Bus Line
-	3400 1550 3800 1550
 Wire Wire Line
 	4000 1300 4000 750
