File: hw/pcb/antenna_side_new/serial_optical_adaptor.sch (KiCad schematic (older format))
At the start: 28 parts, among them IC1 ATMEGA168PA-A, P1 CONN_02X03, P2 Battery, P3 CONN_01X01, P4 CONN_01X04, U1 LM393, U2 LP3984, U3 TXB0108

Commit message: Blas
Parts:
- removed R10, R11, R12: R, Resistors_SMD:R_0805_HandSoldering, symbol R
- C1, C11, C5, C6: value C -> 1u
- C10, C2, C3, C4, C8: value C -> 100n
- C7, C9: value 0.1pF -> 100n
- R4: value R -> 2.7k
Connections:
- wire segments 31 -> 51
Other:
- note removed: "TRANSMITTER"
- moved on the sheet: D2, P4, R1, R2, R3, R4, U1A
